File: kicad/handheld.sch (KiCad schematic (older format))
At the start: 25 parts, among them U1 TLC59025, U10 P-FET, U11 P-FET, U2 74HC595, U3 74HC595, U4 P-FET, U5 P-FET, U6 P-FET, U7 P-FET, U8 P-FET, U9 P-FET

Commit message: Working on schematic
Parts:
- added C? (x2): 100nF, local:C_0805_2012Metric_Pad1.15x1.40mm_widepads, symbol Device:C
- added J?: AVR-PDI-6, symbol Connector:AVR-PDI-6
- added S?: LEFT, digikey-footprints:PushButton_12x12mm_THT_GPTS203211B, symbol dk_Pushbutton-Switches:GPTS203211B
- added S?: RIGHT, digikey-footprints:PushButton_12x12mm_THT_GPTS203211B, symbol dk_Pushbutton-Switches:GPTS203211B
- added S?: SOFTDROP, digikey-footprints:PushButton_12x12mm_THT_GPTS203211B, symbol dk_Pushbutton-Switches:GPTS203211B
- added S?: HARDDROP, digikey-footprints:PushButton_12x12mm_THT_GPTS203211B, symbol dk_Pushbutton-Switches:GPTS203211B
- added S?: ROTL, digikey-footprints:PushButton_12x12mm_THT_GPTS203211B, symbol dk_Pushbutton-Switches:GPTS203211B
- added S?: ROTR, digikey-footprints:PushButton_12x12mm_THT_GPTS203211B, symbol dk_Pushbutton-Switches:GPTS203211B
- added S?: PAUSE, digikey-footprints:PushButton_12x12mm_THT_GPTS203211B, symbol dk_Pushbutton-Switches:GPTS203211B
- added S?: HOLD, digikey-footprints:PushButton_12x12mm_THT_GPTS203211B, symbol dk_Pushbutton-Switches:GPTS203211B
Connections:
- wire segments 317 -> 374
- no-connect marks 11 -> 13
Other:
- moved on the sheet: C3

Commit message: Add datasheets for buck converter and trimmer pot
Parts:
- removed C2, C?: 100nF, local:C_0805_2012Metric_Pad1.15x1.40mm_widepads, symbol Device:C
- removed U2, U3: 74HC595, local:SOIC-16_3.9x9.9mm_P1.27mm_widepads, symbol 74xx:74HC595
- added C4, C5: 100nF, local:C_0805_2012Metric_Pad1.15x1.40mm_widepads, symbol Device:C
- added POT1: 2K TC33X-2-202E, digikey-footprints:Trimpot_3.8mmx3.6mm_TC33X-2-103E, symbol dk_Trimmer-Potentiometers:TC33X-2-103E
- added U12, U3: 74HCT595, symbol 74xx:74HCT595
- R1: value 2.2K -> 1K
- R2: renamed from R?; value 2.2K -> 1K
- gave numbers to parts that had none: 15
Connections:
- wire segments 374 -> 375
- no-connect marks 13 -> 12

Commit message: Move displays to separate sheet
Parts:
- removed D1, D2, D3, D4, D5, D6: DISP_LED_MAT_8x8_COM_ANODE, local:LED_8x8_3MM_38x38MM, symbol akn:DISP_LED_MAT_8x8_COM_ANODE
Connections:
- net labels added: U_PWR
- wire segments 375 -> 284
Other:
- moved on the sheet: C1, C2, C3, C4, C5, C6, J1, R1, R2, U10A, U10B, U11A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

Commit message: Clean up DRC errors and buses
Parts:
- added J1: 61300311121, digikey-footprints:PinHeader_1x3_P2.54_Drill1.1mm, symbol dk_Rectangular-Connectors-Headers-Male-Pins:61300311121
- renumbered C2 to C1, C3 to C2, C1 to C3, J1 to J2, U2 to U1, U8 to U10, U9 to U11, U10 to U12, U11 to U13, U1 to U2, U12 to U4, U13 to U5, U4 to U6, U5 to U7, U6 to U8, U7 to U9
Connections:
- net labels added: COL[0..23], ROW[1..16]
- wire segments 284 -> 257
- no-connect marks 12 -> 43
Other:
- note added: "UART"

Commit message: Change column control to 8 bit bus
Parts:
- removed C6: 100nF, local:C_0805_2012Metric_Pad1.15x1.40mm_widepads, symbol Device:C
- removed POT1: 2K TC33X-2-202E, digikey-footprints:Trimpot_3.8mmx3.6mm_TC33X-2-103E, symbol dk_Trimmer-Potentiometers:TC33X-2-103E
- removed R1, R2: 1K, local:R_1206_3216Metric_Pad1.42x1.75mm_widepads, symbol Device:R
- removed U2, U5: TLC59025, local:SSOP-24_3.9x8.7mm_P0.635mm_widepads, symbol local:TLC59025
- added C4, C7: 100nF, local:C_0805_2012Metric_Pad1.15x1.40mm_widepads, symbol Device:C
- added U10, U13, U16, U19, U25, U28, U3, U31, U34, U46, U49, U6: DMN601, Package_TO_SOT_SMD:SOT-23-6_Handsoldering, symbol local:DMN601
- added U11, U12, U14, U15, U17, U18, U2, U20, U24, U26, U27, U29, U30, U32, U33, U35, U4, U45, U47, U48, U5, U50, U7, U9: NSI45015, digikey-footprints:SOD-123, symbol local:NSI45015
- added U21, U36, U8: SN54LV574, Package_SO:SO-20_5.3x12.6mm_P1.27mm, symbol local:SN54LV574
- renumbered C4 to C5, C5 to C6, U3 to U22, U4 to U23, U6 to U37, U7 to U38, U8 to U39, U9 to U40, U10 to U41, U11 to U42, U12 to U43, U13 to U44
Connections:
- wire segments 257 -> 376
- no-connect marks 43 -> 33

Commit message: Finishes matrix driver circuit
Parts:
- removed C3, C4, C5, C6, C7: 100nF, local:C_0805_2012Metric_Pad1.15x1.40mm_widepads, symbol Device:C
- removed U10, U13, U16, U19, U25, U28, U3, U31, U34, U46, U49, U6: DMN601, Package_TO_SOT_SMD:SOT-23-6_Handsoldering, symbol local:DMN601
- removed U11, U12, U14, U15, U17, U18, U2, U20, U24, U26, U27, U29, U30, U32, U33, U35, U4, U45, U47, U48, U5, U50, U7, U9: NSI45015, digikey-footprints:SOD-123, symbol local:NSI45015
- removed U21, U36, U8: SN54LV574, Package_SO:SO-20_5.3x12.6mm_P1.27mm, symbol local:SN54LV574
- removed U22, U23: 74HCT595, symbol 74xx:74HCT595
- removed U37, U38, U39, U40, U41, U42, U43, U44: P-FET, local:SOIC-8_3.9x4.9mm_P1.27mm_widepads, symbol local:P-FET
Connections:
- net labels removed: COL0, COL1, COL10, COL11, COL12, COL13, COL14, COL15, COL16, COL17, COL18, COL19, COL2, COL20, COL21, COL22, COL23, COL3, COL4, COL5, COL6, COL7, COL8, COL9, COL[0..23], ROW1, ROW10, ROW11, ROW12, ROW13, ROW14, ROW15, ROW16, ROW2, ROW3, ROW4, ROW5, ROW6, ROW7, ROW8, ROW9, ROW[1..16]
- wire segments 376 -> 63
- no-connect marks 33 -> 16

Commit message: Switches to ATXMEGA64C3 for USB
Parts:
- added U1: ATxmega64C3-AU, Package_QFP:TQFP-64_14x14mm_P0.8mm, symbol MCU_Microchip_ATmega:ATxmega64C3-AU
- renumbered U1 to U2
Connections:
- net labels added: D+, D-, D0, D1, D2, D3, D4, D5, D6, D7, D[0..7], RX, TX
- wire segments 63 -> 73
- no-connect marks 16 -> 6
Other:
- moved on the sheet: C1, C2, J1, J2

Commit message: Adds IrDA transceiver
Parts:
- removed U2: ATxmega64D4-AU, Package_QFP:TQFP-44_10x10mm_P0.8mm, symbol MCU_Microchip_ATmega:ATxmega64D4-AU
- added C1: 100nF, local:C_0805_2012Metric_Pad1.15x1.40mm_widepads, symbol Device:C
- added R1: 47R, symbol Device:R
- added U1: TFBS4711, local:FPC_6, symbol local:TFBS4711
- renumbered C1 to C2, C2 to C3, U1 to U2
Connections:
- net labels removed: COLCLK, COLSDI0, COLSDI16, LE, ROWCLK, ROWSDI, ~OE
- wire segments 73 -> 96
Other:
- moved on the sheet: C2, C3, J1, J2, U2
