File: kicad/handheld.sch (KiCad schematic (older format))
At the start: 16 parts, among them J1 61300311121, J2 AVR-PDI-6, U1 TFBS4711, U2 ATxmega64C3-AU

Commit message: Adds piezo buzzer
Parts:
- added BZ?: PS1240P02BT, digikey-footprints:Piezo_Transducer_THT_PS1240P02BT, symbol dk_Alarms-Buzzers-and-Sirens:PS1240P02BT
- added RV?: 2K, symbol Device:R_POT
Connections:
- wire segments 96 -> 98
Other:
- moved on the sheet: C1, R1, U1
Changed lines of the file:
@@
 L local:TFBS4711 U1
 U 1 1 610B6C7F
-P 1100 2875
-F 0 "U1" H 1067 3400 50  0000 C CNN
-F 1 "TFBS4711" H 1067 3309 50  0000 C CNN
-F 2 "local:FPC_6" H 1150 2975 50  0001 C CNN
-F 3 "https://www.vishay.com/docs/82633/tfbs4711.pdf" H 1150 2975 50  0001 C CNN
-	1    1100 2875
+P 1100 2325
+F 0 "U1" H 1067 2850 50  0000 C CNN
+F 1 "TFBS4711" H 1067 2759 50  0000 C CNN
+F 2 "local:FPC_6" H 1150 2425 50  0001 C CNN
+F 3 "https://www.vishay.com/docs/82633/tfbs4711.pdf" H 1150 2425 50  0001 C CNN
+	1    1100 2325
 	-1   0    0    -1
 $EndComp
@@
 L power:GND #PWR02
 U 1 1 610B848D
-P 1600 3375
-F 0 "#PWR02" H 1600 3125 50  0001 C CNN
-F 1 "GND" V 1605 3247 50  0000 R CNN
-F 2 "" H 1600 3375 50  0001 C CNN
-F 3 "" H 1600 3375 50  0001 C CNN
-	1    1600 3375
+P 1600 2825
+F 0 "#PWR02" H 1600 2575 50  0001 C CNN
+F 1 "GND" V 1605 2697 50  0000 R CNN
+F 2 "" H 1600 2825 50  0001 C CNN
+F 3 "" H 1600 2825 50  0001 C CNN
+	1    1600 2825
 	1    0    0    -1
 $EndComp
-Text GLabel 2075 3075 2    50   Input ~ 0
+Text GLabel 2075 2525 2    50   Input ~ 0
 VDD
 Wire Wire Line
@@
 L Device:R R1
 U 1 1 610D52DA
-P 1825 3075
-F 0 "R1" V 1750 3075 50  0000 C CNN
-F 1 "47R" V 1825 3075 50  0000 C CNN
-F 2 "" V 1755 3075 50  0001 C CNN
-F 3 "~" H 1825 3075 50  0001 C CNN
-	1    1825 3075
+P 1825 2525
+F 0 "R1" V 1750 2525 50  0000 C CNN
+F 1 "47R" V 1825 2525 50  0000 C CNN
+F 2 "" V 1755 2525 50  0001 C CNN
+F 3 "~" H 1825 2525 50  0001 C CNN
+	1    1825 2525
 	0    1    1    0
 $EndComp
@@
 L Device:C C1
 U 1 1 610DC121
-P 1600 3225
-F 0 "C1" V 1375 3250 50  0000 C CNN
-F 1 "100nF" V 1450 3275 50  0000 C CNN
-F 2 "local:C_0805_2012Metric_Pad1.15x1.40mm_widepads" H 1638 3075 50  0001 C CNN
-F 3 "~" H 1600 3225 50  0001 C CNN
-	1    1600 3225
+P 1600 2675
+F 0 "C1" V 1375 2700 50  0000 C CNN
+F 1 "100nF" V 1450 2725 50  0000 C CNN
+F 2 "local:C_0805_2012Metric_Pad1.15x1.40mm_widepads" H 1638 2525 50  0001 C CNN
+F 3 "~" H 1600 2675 50  0001 C CNN
+	1    1600 2675
 	-1   0    0    1
 $EndComp
 Wire Wire Line
-	1400 3375 1600 3375
+	1400 2825 1600 2825
 Wire Wire Line
-	1400 3175 1400 3375
-Connection ~ 1600 3375
+	1400 2625 1400 2825
+Connection ~ 1600 2825
 Wire Wire Line
-	1400 3075 1600 3075
-Connection ~ 1600 3075
+	1400 2525 1600 2525
+Connection ~ 1600 2525
 Wire Wire Line
-	1600 3075 1675 3075
+	1600 2525 1675 2525
 Wire Wire Line
-	1400 2875 2625 2875
+	1400 2325 2625 2325
 Wire Wire Line
-	2625 2875 2625 4375
+	2625 2325 2625 4375
 Wire Wire Line
-	1400 2775 2700 2775
+	1400 2225 2700 2225
 Wire Wire Line
-	2700 2775 2700 4175
+	2700 2225 2700 4175
 Wire Wire Line
-	1400 2675 2775 2675
+	1400 2125 2775 2125
 Wire Wire Line
-	2775 2675 2775 4075
+	2775 2125 2775 4075
 Wire Wire Line
-	1975 3075 2075 3075
-Text GLabel 1650 2575 2    50   UnSpc ~ 0
+	1975 2525 2075 2525
+Text GLabel 1650 2025 2    50   UnSpc ~ 0
 U_PWR
 Wire Wire Line
-	1400 2575 1650 2575
+	1400 2025 1650 2025
+$Comp
+L dk_Alarms-Buzzers-and-Sirens:PS1240P02BT BZ?
+U 1 1 5F87649F
+P 1225 3325
+F 0 "BZ?" H 1323 3078 60  0000 C CNN
+F 1 "PS1240P02BT" H 1323 3184 60  0000 C CNN
+F 2 "digikey-footprints:Piezo_Transducer_THT_PS1240P02BT" H 1425 3525 60  0001 L CNN
+F 3 "https://product.tdk.com/info/en/catalog/datasheets/piezoelectronic_buzzer_ps_en.pdf" H 1425 3625 60  0001 L CNN
+F 4 "445-2525-1-ND" H 1425 3725 60  0001 L CNN "Digi-Key_PN"
+F 5 "PS1240P02BT" H 1425 3825 60  0001 L CNN "MPN"
+F 6 "Audio Products" H 1425 3925 60  0001 L CNN "Category"
+F 7 "Alarms, Buzzers, and Sirens" H 1425 4025 60  0001 L CNN "Family"
+F 8 "https://product.tdk.com/info/en/catalog/datasheets/piezoelectronic_buzzer_ps_en.pdf" H 1425 4125 60  0001 L CNN "DK_Datasheet_Link"
+F 9 "/product-detail/en/tdk-corporation/PS1240P02BT/445-2525-1-ND/935930" H 1425 4225 60  0001 L CNN "DK_Detail_Page"
+F 10 "AUDIO PIEZO TRANSDUCER 30V TH" H 1425 4325 60  0001 L CNN "Description"
+F 11 "TDK Corporation" H 1425 4425 60  0001 L CNN "Manufacturer"
+F 12 "Active" H 1425 4525 60  0001 L CNN "Status"
+	1    1225 3325
+	-1   0    0    1
+$EndComp
+Wire Wire Line
+	2200 3475 3750 3475
+$Comp
+L Device:R_POT RV?
+U 1 1 5F890273
+P 2200 3325
+F 0 "RV?" H 2130 3279 50  0000 R CNN
+F 1 "2K" H 2130 3370 50  0000 R CNN
+F 2 "" H 2200 3325 50  0001 C CNN
+F 3 "~" H 2200 3325 50  0001 C CNN
+	1    2200 3325
+	-1   0    0    1
+$EndComp
+$Comp
+L power:GND #PWR?
+U 1 1 5F89CA0B
+P 2200 3175
+F 0 "#PWR?" H 2200 2925 50  0001 C CNN
+F 1 "GND" V 2205 3047 50  0000 R CNN
+F 2 "" H 2200 3175 50  0001 C CNN
+F 3 "" H 2200 3175 50  0001 C CNN
+	1    2200 3175
+	-1   0    0    1
+$EndComp
+Wire Wire Line
+	1325 3325 2050 3325
 Wire Bus Line
 	5775 4875 5775 5175
 Wire Bus Line
 	5775 4475 5775 4875
+$Comp
+L power:GND #PWR?
+U 1 1 5F8A383B
+P 1325 3425
+F 0 "#PWR?" H 1325 3175 50  0001 C CNN
+F 1 "GND" V 1330 3297 50  0000 R CNN
+F 2 "" H 1325 3425 50  0001 C CNN
+F 3 "" H 1325 3425 50  0001 C CNN
+	1    1325 3425
+	0    -1   -1   0
+$EndComp
 $EndSCHEMATC

Commit message: Adds GPIO expansion port
Parts:
- added C2: 4.7uF, local:C_0805_2012Metric_Pad1.15x1.40mm_widepads, symbol Device:C
- added J1: Conn_01x08, symbol Connector_Generic:Conn_01x08
- added R1: R_PHOTO, symbol Device:R_PHOTO
- added R3: 10K, symbol Device:R
- added RV1: 100R, symbol Device:R_POT
- gave numbers to parts that had none: 2
- renumbered C2 to C3, C3 to C4, J1 to J2, J2 to J3, R1 to R2
Connections:
- wire segments 98 -> 136
- no-connect marks 6 -> 11
Other:
- note added: "GPIO Expansion"

Commit message: Adds AA battery holders
Parts:
- C1, C2, C3, C4: footprint local:C_0805_2012Metric_Pad1.15x1.40mm_widepads -> Capacitor_SMD:C_0805_2012Metric_Pad1.15x1.40mm_HandSolder
- J1: footprint (none) -> Connector_PinSocket_2.00mm:PinSocket_1x08_P2.00mm_Horizontal
- R2, R3, RV1, RV2: footprint (none) -> Resistor_SMD:R_0805_2012Metric_Pad1.15x1.40mm_HandSolder
Changed lines of the file:
@@
 F 0 "C4" V 4348 6675 50  0000 C CNN
 F 1 "100nF" V 4439 6675 50  0000 C CNN
-F 2 "local:C_0805_2012Metric_Pad1.15x1.40mm_widepads" H 4638 6525 50  0001 C CNN
+F 2 "Capacitor_SMD:C_0805_2012Metric_Pad1.15x1.40mm_HandSolder" H 4638 6525 50  0001 C CNN
 F 3 "~" H 4600 6675 50  0001 C CNN
 	1    4600 6675
@@
 F 0 "C3" V 3948 6675 50  0000 C CNN
 F 1 "100nF" V 4039 6675 50  0000 C CNN
-F 2 "local:C_0805_2012Metric_Pad1.15x1.40mm_widepads" H 4238 6525 50  0001 C CNN
+F 2 "Capacitor_SMD:C_0805_2012Metric_Pad1.15x1.40mm_HandSolder" H 4238 6525 50  0001 C CNN
 F 3 "~" H 4200 6675 50  0001 C CNN
 	1    4200 6675
@@
 F 0 "R2" V 1750 2525 50  0000 C CNN
 F 1 "47R" V 1825 2525 50  0000 C CNN
-F 2 "" V 1755 2525 50  0001 C CNN
+F 2 "Resistor_SMD:R_0805_2012Metric_Pad1.15x1.40mm_HandSolder" V 1755 2525 50  0001 C CNN
 F 3 "~" H 1825 2525 50  0001 C CNN
 	1    1825 2525
@@
 F 0 "C1" V 1375 2700 50  0000 C CNN
 F 1 "100nF" V 1450 2725 50  0000 C CNN
-F 2 "local:C_0805_2012Metric_Pad1.15x1.40mm_widepads" H 1638 2525 50  0001 C CNN
+F 2 "Capacitor_SMD:C_0805_2012Metric_Pad1.15x1.40mm_HandSolder" H 1638 2525 50  0001 C CNN
 F 3 "~" H 1600 2675 50  0001 C CNN
 	1    1600 2675
@@
 F 0 "RV2" H 2130 3371 50  0000 R CNN
 F 1 "2K" H 2130 3280 50  0000 R CNN
-F 2 "" H 2200 3325 50  0001 C CNN
+F 2 "Resistor_SMD:R_0805_2012Metric_Pad1.15x1.40mm_HandSolder" H 2200 3325 50  0001 C CNN
 F 3 "~" H 2200 3325 50  0001 C CNN
 	1    2200 3325
@@
 F 0 "R3" V 1843 6225 50  0000 C CNN
 F 1 "10K" V 1934 6225 50  0000 C CNN
-F 2 "" V 1980 6225 50  0001 C CNN
+F 2 "Resistor_SMD:R_0805_2012Metric_Pad1.15x1.40mm_HandSolder" V 1980 6225 50  0001 C CNN
 F 3 "~" H 2050 6225 50  0001 C CNN
 	1    2050 6225
@@
 F 0 "RV1" V 1343 1500 50  0000 C CNN
 F 1 "100R" V 1434 1500 50  0000 C CNN
-F 2 "" H 1550 1500 50  0001 C CNN
+F 2 "Resistor_SMD:R_0805_2012Metric_Pad1.15x1.40mm_HandSolder" H 1550 1500 50  0001 C CNN
 F 3 "~" H 1550 1500 50  0001 C CNN
 	1    1550 1500
@@
 F 0 "C2" V 2075 1350 50  0000 C CNN
 F 1 "4.7uF" V 2000 1175 50  0000 C CNN
-F 2 "local:C_0805_2012Metric_Pad1.15x1.40mm_widepads" H 1963 1200 50  0001 C CNN
+F 2 "Capacitor_SMD:C_0805_2012Metric_Pad1.15x1.40mm_HandSolder" H 1963 1200 50  0001 C CNN
 F 3 "~" H 1925 1350 50  0001 C CNN
 	1    1925 1350
@@
 F 0 "J1" V 2972 7305 50  0000 L CNN
 F 1 "Conn_01x08" V 3063 7305 50  0000 L CNN
-F 2 "" H 3100 6925 50  0001 C CNN
+F 2 "Connector_PinSocket_2.00mm:PinSocket_1x08_P2.00mm_Horizontal" H 3100 6925 50  0001 C CNN
 F 3 "~" H 3100 6925 50  0001 C CNN
 	1    3100 6925

Commit message: Adds AVR/PDI header footprint
Parts:
- removed S1: HOLD, digikey-footprints:PushButton_12x12mm_THT_GPTS203211B, symbol dk_Pushbutton-Switches:GPTS203211B
- removed S2: PAUSE, digikey-footprints:PushButton_12x12mm_THT_GPTS203211B, symbol dk_Pushbutton-Switches:GPTS203211B
- removed S3: ROTR, digikey-footprints:PushButton_12x12mm_THT_GPTS203211B, symbol dk_Pushbutton-Switches:GPTS203211B
- removed S4: ROTL, digikey-footprints:PushButton_12x12mm_THT_GPTS203211B, symbol dk_Pushbutton-Switches:GPTS203211B
- removed S5: HARDDROP, digikey-footprints:PushButton_12x12mm_THT_GPTS203211B, symbol dk_Pushbutton-Switches:GPTS203211B
- removed S6: SOFTDROP, digikey-footprints:PushButton_12x12mm_THT_GPTS203211B, symbol dk_Pushbutton-Switches:GPTS203211B
- removed S7: RIGHT, digikey-footprints:PushButton_12x12mm_THT_GPTS203211B, symbol dk_Pushbutton-Switches:GPTS203211B
- removed S8: LEFT, digikey-footprints:PushButton_12x12mm_THT_GPTS203211B, symbol dk_Pushbutton-Switches:GPTS203211B
- added SW1: HOLD, Button_Switch_THT:SW_PUSH-12mm, symbol Switch:SW_Push
- added SW2: PAUSE, Button_Switch_THT:SW_PUSH-12mm, symbol Switch:SW_Push
- added SW3: SDROP, Button_Switch_THT:SW_PUSH-12mm, symbol Switch:SW_Push
- added SW4: HDROP, Button_Switch_THT:SW_PUSH-12mm, symbol Switch:SW_Push
- added SW5: ROTR, Button_Switch_THT:SW_PUSH-12mm, symbol Switch:SW_Push
- added SW6, SW8: RIGHT, Button_Switch_THT:SW_PUSH-12mm, symbol Switch:SW_Push
- added SW7: ROTL, Button_Switch_THT:SW_PUSH-12mm, symbol Switch:SW_Push
- J3: footprint (none) -> local:AVR_PDI_Header_2x03_P2.54mm_Vertical
- R1: footprint (none) -> OptoDevice:R_LDR_5.1x4.3mm_P3.4mm_Vertical
Connections:
- wire segments 136 -> 141

Commit message: Fixes footprints
Parts:
- RV1, RV2: footprint Resistor_SMD:R_0805_2012Metric_Pad1.15x1.40mm_HandSolder -> Potentiometer_SMD:Potentiometer_Bourns_TC33X_Vertical
- U1: footprint local:FPC_6 -> local:TFBS4711-IrDA
Changed lines of the file:
@@
 F 0 "U1" H 1067 2850 50  0000 C CNN
 F 1 "TFBS4711" H 1067 2759 50  0000 C CNN
-F 2 "local:FPC_6" H 1150 2425 50  0001 C CNN
+F 2 "local:TFBS4711-IrDA" H 1150 2425 50  0001 C CNN
 F 3 "https://www.vishay.com/docs/82633/tfbs4711.pdf" H 1150 2425 50  0001 C CNN
 	1    1100 2325
@@
 F 0 "RV2" H 2130 3371 50  0000 R CNN
 F 1 "2K" H 2130 3280 50  0000 R CNN
-F 2 "Resistor_SMD:R_0805_2012Metric_Pad1.15x1.40mm_HandSolder" H 2200 3325 50  0001 C CNN
+F 2 "Potentiometer_SMD:Potentiometer_Bourns_TC33X_Vertical" H 2200 3325 50  0001 C CNN
 F 3 "~" H 2200 3325 50  0001 C CNN
 	1    2200 3325
@@
 F 0 "RV1" V 1343 1500 50  0000 C CNN
 F 1 "100R" V 1434 1500 50  0000 C CNN
-F 2 "Resistor_SMD:R_0805_2012Metric_Pad1.15x1.40mm_HandSolder" H 1550 1500 50  0001 C CNN
+F 2 "Potentiometer_SMD:Potentiometer_Bourns_TC33X_Vertical" H 1550 1500 50  0001 C CNN
 F 3 "~" H 1550 1500 50  0001 C CNN
 	1    1550 1500

Commit message: Adds column drivers
Parts:
- J1: footprint Connector_PinSocket_2.00mm:PinSocket_1x08_P2.00mm_Horizontal -> Connector_PinSocket_2.54mm:PinSocket_1x08_P2.54mm_Horizontal
- J2: footprint digikey-footprints:PinHeader_1x3_P2.54_Drill1.1mm -> Connector_PinSocket_2.54mm:PinSocket_1x03_P2.54mm_Horizontal
Changed lines of the file:
@@
 F 0 "J2" V 3200 3075 50  0000 R CNN
 F 1 "61300311121" H 3550 2875 50  0000 R CNN
-F 2 "digikey-footprints:PinHeader_1x3_P2.54_Drill1.1mm" H 3525 3275 60  0001 L CNN
+F 2 "Connector_PinSocket_2.54mm:PinSocket_1x03_P2.54mm_Horizontal" H 3525 3275 60  0001 L CNN
 F 3 "https://katalog.we-online.de/em/datasheet/6130xx11121.pdf" H 3525 3375 60  0001 L CNN
 F 4 "732-5316-ND" H 3525 3475 60  0001 L CNN "Digi-Key_PN"
@@
 F 0 "J1" V 2972 7305 50  0000 L CNN
 F 1 "Conn_01x08" V 3063 7305 50  0000 L CNN
-F 2 "Connector_PinSocket_2.00mm:PinSocket_1x08_P2.00mm_Horizontal" H 3100 6925 50  0001 C CNN
+F 2 "Connector_PinSocket_2.54mm:PinSocket_1x08_P2.54mm_Horizontal" H 3100 6925 50  0001 C CNN
 F 3 "~" H 3100 6925 50  0001 C CNN
 	1    3100 6925
