File: kicad/power.sch (KiCad schematic (older format))
At the start: 10 parts, among them J2 UE27AC54100, U14 P-FET, U15 LM3671MF-3.3

Commit message: Move displays to separate sheet
Parts:
- added BT?: 2 x 1.5V AA, symbol Device:Battery
- added R?: 100K, symbol Device:R
- BT1: value 4 x 1.5V AA -> 2 x 1.5V AA
- R3: value 100K -> 10K
Connections:
- net labels added: 3.5-5V, BAT_LVL, U_PWR
- wire segments 39 -> 47
Other:
- note added: "Unregulated power directly from USB or\nbatteries. Ranges between 3.5 and 5V.\nDriving LEDs with constant current drivers."
- moved on the sheet: BT1
Changed lines of the file:
@@
 $Descr A4 11693 8268
 encoding utf-8
-Sheet 2 2
+Sheet 2 3
 Title ""
 Date ""
@@
 Wire Wire Line
 	5500 3850 5500 3975
-Text GLabel 7325 3450 2    50   Input ~ 0
-VDD
 Connection ~ 6725 3450
 $Comp
 L Device:Battery BT1
 U 1 1 5F7915DC
-P 2400 3725
-F 0 "BT1" H 2125 3800 50  0000 L CNN
-F 1 "4 x 1.5V AA" H 1825 3650 50  0000 L CNN
-F 2 "" V 2400 3785 50  0001 C CNN
-F 3 "~" V 2400 3785 50  0001 C CNN
-	1    2400 3725
-	1    0    0    -1
+P 2075 3450
+F 0 "BT1" V 1925 3375 50  0000 L CNN
+F 1 "2 x 1.5V AA" V 2225 3225 50  0000 L CNN
+F 2 "" V 2075 3510 50  0001 C CNN
+F 3 "~" V 2075 3510 50  0001 C CNN
+	1    2075 3450
+	0    1    -1   0
 $EndComp
 Wire Wire Line
 	4225 3450 4300 3450
 Connection ~ 4300 3450
-Text Label 2400 3450 0    50   ~ 0
+Text Label 2475 3450 2    50   ~ 0
 6V
 $Comp
@@
 $EndComp
 Wire Wire Line
-	3625 3450 3200 3450
+	3625 3450 3400 3450
 Wire Wire Line
 	4225 3550 4300 3550
@@
 P 3525 3825
 F 0 "R3" H 3595 3871 50  0000 L CNN
-F 1 "100K" H 3595 3780 50  0000 L CNN
+F 1 "10K" H 3595 3780 50  0000 L CNN
 F 2 "" V 3455 3825 50  0001 C CNN
 F 3 "~" H 3525 3825 50  0001 C CNN
@@
 	1    0    0    -1
 $EndComp
-Connection ~ 3525 3975
 Wire Wire Line
 	3525 3675 3525 3550
@@
 L pspice:DIODE D7
 U 1 1 5F8CC172
-P 3000 3450
-F 0 "D7" H 3000 3715 50  0000 C CNN
-F 1 "1N4007" H 3000 3624 50  0000 C CNN
-F 2 "" H 3000 3450 50  0001 C CNN
-F 3 "~" H 3000 3450 50  0001 C CNN
-	1    3000 3450
-	1    0    0    -1
-$EndComp
-Wire Wire Line
-	2800 3450 2400 3450
-Wire Wire Line
-	2400 3450 2400 3525
-Wire Wire Line
-	2400 3975 2400 3925
-Wire Wire Line
-	2400 3975 3525 3975
+P 3200 3450
+F 0 "D7" H 3200 3715 50  0000 C CNN
+F 1 "1N4007" H 3200 3624 50  0000 C CNN
+F 2 "" H 3200 3450 50  0001 C CNN
+F 3 "~" H 3200 3450 50  0001 C CNN
+	1    3200 3450
+	1    0    0    -1
+$EndComp
+Wire Wire Line
+	1825 3450 1875 3450
 Wire Wire Line
 	4925 3600 4925 3450
@@
 U 1 1 5F789842
 P 4925 3750
-F 0 "C7" H 4650 3800 50  0000 L CNN
-F 1 "4.7uF" H 4575 3650 50  0000 L CNN
+F 0 "C7" H 4725 3750 50  0000 L CNN
+F 1 "4.7uF" H 4700 3650 50  0000 L CNN
 F 2 "" H 4963 3600 50  0001 C CNN
 F 3 "~" H 4925 3750 50  0001 C CNN
@@
 Connection ~ 4925 3450
 Wire Wire Line
-	4925 3450 4300 3450
+	4925 3450 4575 3450
 Connection ~ 4925 3975
 Wire Wire Line
-	4925 3975 5500 3975
+	4925 3975 5150 3975
 Wire Wire Line
 	3825 2200 3825 2375
@@
 	4300 2825 4300 3450
 Wire Wire Line
-	5200 3550 5075 3550
+	5200 3550 5150 3550
 Wire Wire Line
 	5075 3550 5075 3450
@@
 	1    0    0    -1
 $EndComp
+$Comp
+L Device:R R?
+U 1 1 5F2BAEAD
+P 5150 3825
+F 0 "R?" H 5220 3871 50  0000 L CNN
+F 1 "100K" H 5220 3780 50  0000 L CNN
+F 2 "" V 5080 3825 50  0001 C CNN
+F 3 "~" H 5150 3825 50  0001 C CNN
+	1    5150 3825
+	1    0    0    -1
+$EndComp
+Connection ~ 5150 3975
+Wire Wire Line
+	5150 3975 5500 3975
+Wire Wire Line
+	5150 3675 5150 3550
+Connection ~ 5150 3550
+Wire Wire Line
+	5150 3550 5075 3550
+Wire Wire Line
+	4575 3450 4575 3025
+Wire Wire Line
+	4575 3025 7325 3025
+Connection ~ 4575 3450
+Wire Wire Line
+	4575 3450 4300 3450
+Text Label 7000 3025 0    50   ~ 0
+3.5-5V
+Text Notes 5275 3025 0    50   ~ 0
+Unregulated power directly from USB or\nbatteries. Ranges between 3.5 and 5V.\nDriving LEDs with constant current drivers.
+$Comp
+L Device:Battery BT?
+U 1 1 5F45FF3D
+P 2075 3975
+F 0 "BT?" V 1925 3925 50  0000 L CNN
+F 1 "2 x 1.5V AA" V 2225 3750 50  0000 L CNN
+F 2 "" V 2075 4035 50  0001 C CNN
+F 3 "~" V 2075 4035 50  0001 C CNN
+	1    2075 3975
+	0    -1   1    0
+$EndComp
+Wire Wire Line
+	2275 3975 3525 3975
+Wire Wire Line
+	1875 3975 1825 3975
+Text HLabel 1825 2925 2    50   Output ~ 0
+BAT_LVL
+Wire Wire Line
+	1825 3975 1825 3450
+Connection ~ 3525 3975
+Wire Wire Line
+	2275 3450 3000 3450
+Wire Wire Line
+	1825 3450 1825 2925
+Connection ~ 1825 3450
+Text HLabel 7325 3025 2    50   Output ~ 0
+U_PWR
+Text HLabel 7325 3450 2    50   Output ~ 0
+VDD
 $EndSCHEMATC

Commit message: Clean up DRC errors and buses
Parts:
- gave numbers to parts that had none: 2
- renumbered D7 to D1, D8 to D2, J2 to J3
Connections:
- wire segments 47 -> 45
- no-connect marks 2 -> 3
Changed lines of the file:
@@
 	6475 3450 6725 3450
 $Comp
-L power:GND #PWR020
+L power:GND #PWR022
 U 1 1 5F78F1EA
 P 5500 3975
-F 0 "#PWR020" H 5500 3725 50  0001 C CNN
+F 0 "#PWR022" H 5500 3725 50  0001 C CNN
 F 1 "GND" H 5505 3802 50  0000 C CNN
 F 2 "" H 5500 3975 50  0001 C CNN
@@
 6V
 $Comp
-L power:PWR_FLAG #FLG02
-U 1 1 5F793D23
-P 6725 3450
-F 0 "#FLG02" H 6725 3525 50  0001 C CNN
-F 1 "PWR_FLAG" H 6725 3623 50  0000 C CNN
-F 2 "" H 6725 3450 50  0001 C CNN
-F 3 "~" H 6725 3450 50  0001 C CNN
-	1    6725 3450
-	1    0    0    -1
-$EndComp
-$Comp
 L power:PWR_FLAG #FLG01
 U 1 1 5F794155
@@
 	6275 3975 6725 3975
 $Comp
-L dk_USB-DVI-HDMI-Connectors:UE27AC54100 J2
+L dk_USB-DVI-HDMI-Connectors:UE27AC54100 J3
 U 1 1 5F8B701D
 P 3625 1900
-F 0 "J2" V 3692 2253 60  0000 L CNN
+F 0 "J3" V 3692 2253 60  0000 L CNN
 F 1 "UE27AC54100" V 3798 2253 60  0000 L CNN
 F 2 "digikey-footprints:USB_A_Female_UE27AC54100" H 3825 2100 60  0001 L CNN
@@
 Wire Wire Line
 	3625 3450 3400 3450
-Wire Wire Line
-	4225 3550 4300 3550
-Wire Wire Line
-	4300 3550 4300 3450
 $Comp
 L Device:R R3
@@
 NoConn ~ 3725 2200
 $Comp
-L pspice:DIODE D7
+L pspice:DIODE D1
 U 1 1 5F8CC172
 P 3200 3450
-F 0 "D7" H 3200 3715 50  0000 C CNN
+F 0 "D1" H 3200 3715 50  0000 C CNN
 F 1 "1N4007" H 3200 3624 50  0000 C CNN
 F 2 "" H 3200 3450 50  0001 C CNN
@@
 $EndComp
 Connection ~ 4925 3450
-Wire Wire Line
-	4925 3450 4575 3450
 Connection ~ 4925 3975
 Wire Wire Line
@@
 Connection ~ 3525 3550
 $Comp
-L pspice:DIODE D8
+L pspice:DIODE D2
 U 1 1 5F8D97D5
 P 3950 2825
-F 0 "D8" H 3950 3090 50  0000 C CNN
+F 0 "D2" H 3950 3090 50  0000 C CNN
 F 1 "1N4007" H 3950 2999 50  0000 C CNN
 F 2 "" H 3950 2825 50  0001 C CNN
@@
 	5075 3450 4925 3450
 $Comp
-L power:GND #PWR?
+L power:GND #PWR021
 U 1 1 5F8DC955
 P 3300 2025
-F 0 "#PWR?" H 3300 1775 50  0001 C CNN
+F 0 "#PWR021" H 3300 1775 50  0001 C CNN
 F 1 "GND" H 3305 1852 50  0000 C CNN
 F 2 "" H 3300 2025 50  0001 C CNN
@@
 $EndComp
 $Comp
-L Device:R R?
+L Device:R R4
 U 1 1 5F2BAEAD
 P 5150 3825
-F 0 "R?" H 5220 3871 50  0000 L CNN
+F 0 "R4" H 5220 3871 50  0000 L CNN
 F 1 "100K" H 5220 3780 50  0000 L CNN
 F 2 "" V 5080 3825 50  0001 C CNN
@@
 Unregulated power directly from USB or\nbatteries. Ranges between 3.5 and 5V.\nDriving LEDs with constant current drivers.
 $Comp
-L Device:Battery BT?
+L Device:Battery BT2
 U 1 1 5F45FF3D
 P 2075 3975
-F 0 "BT?" V 1925 3925 50  0000 L CNN
+F 0 "BT2" V 1925 3925 50  0000 L CNN
 F 1 "2 x 1.5V AA" V 2225 3750 50  0000 L CNN
 F 2 "" V 2075 4035 50  0001 C CNN
@@
 	1825 3450 1825 2925
 Connection ~ 1825 3450
-Text HLabel 7325 3025 2    50   Output ~ 0
+Text HLabel 7325 3025 2    50   UnSpc ~ 0
 U_PWR
 Text HLabel 7325 3450 2    50   Output ~ 0
 VDD
+Wire Wire Line
+	4575 3450 4925 3450
+NoConn ~ 4225 3550
 $EndSCHEMATC

Commit message: Change column control to 8 bit bus
Parts:
- renumbered C7 to C8, C8 to C9, R3 to R1, R4 to R2, U14 to U51, U15 to U52
Changed lines of the file:
@@
 $EndDescr
 $Comp
-L Regulator_Switching:LM3670MF U15
+L Regulator_Switching:LM3670MF U52
 U 1 1 5F788F1B
 P 5500 3550
-F 0 "U15" H 5500 3875 50  0000 C CNN
+F 0 "U52" H 5500 3875 50  0000 C CNN
 F 1 "LM3671MF-3.3" H 5500 3784 50  0000 C CNN
 F 2 "Package_TO_SOT_SMD:TSOT-23-5" H 5550 3300 50  0001 L CNN
@@
 	5200 3450 5075 3450
 $Comp
-L Device:C C8
+L Device:C C9
 U 1 1 5F78C119
 P 6725 3750
-F 0 "C8" H 6840 3796 50  0000 L CNN
+F 0 "C9" H 6840 3796 50  0000 L CNN
 F 1 "10uF" H 6840 3705 50  0000 L CNN
 F 2 "" H 6763 3600 50  0001 C CNN
@@
 	6475 3450 6725 3450
 $Comp
-L power:GND #PWR022
+L power:GND #PWR020
 U 1 1 5F78F1EA
 P 5500 3975
-F 0 "#PWR022" H 5500 3725 50  0001 C CNN
+F 0 "#PWR020" H 5500 3725 50  0001 C CNN
 F 1 "GND" H 5505 3802 50  0000 C CNN
 F 2 "" H 5500 3975 50  0001 C CNN
@@
 $EndComp
 $Comp
-L local:P-FET U14
+L local:P-FET U51
 U 1 1 5F8BAAF4
 P 3925 3500
-F 0 "U14" H 3925 3815 50  0000 C CNN
+F 0 "U51" H 3925 3815 50  0000 C CNN
 F 1 "P-FET" H 3925 3724 50  0000 C CNN
 F 2 "" H 4125 3900 50  0001 C CNN
@@
 	3625 3450 3400 3450
 $Comp
-L Device:R R3
+L Device:R R1
 U 1 1 5F8BFEFE
 P 3525 3825
-F 0 "R3" H 3595 3871 50  0000 L CNN
+F 0 "R1" H 3595 3871 50  0000 L CNN
 F 1 "10K" H 3595 3780 50  0000 L CNN
 F 2 "" V 3455 3825 50  0001 C CNN
@@
 	4925 3900 4925 3975
 $Comp
-L Device:C C7
+L Device:C C8
 U 1 1 5F789842
 P 4925 3750
-F 0 "C7" H 4725 3750 50  0000 L CNN
+F 0 "C8" H 4725 3750 50  0000 L CNN
 F 1 "4.7uF" H 4700 3650 50  0000 L CNN
 F 2 "" H 4963 3600 50  0001 C CNN
@@
 	5075 3450 4925 3450
 $Comp
-L power:GND #PWR021
+L power:GND #PWR019
 U 1 1 5F8DC955
 P 3300 2025
-F 0 "#PWR021" H 3300 1775 50  0001 C CNN
+F 0 "#PWR019" H 3300 1775 50  0001 C CNN
 F 1 "GND" H 3305 1852 50  0000 C CNN
 F 2 "" H 3300 2025 50  0001 C CNN
@@
 $EndComp
 $Comp
-L Device:R R4
+L Device:R R2
 U 1 1 5F2BAEAD
 P 5150 3825
-F 0 "R4" H 5220 3871 50  0000 L CNN
+F 0 "R2" H 5220 3871 50  0000 L CNN
 F 1 "100K" H 5220 3780 50  0000 L CNN
 F 2 "" V 5080 3825 50  0001 C CNN

Commit message: Switches to ATXMEGA64C3 for USB
Parts:
- renumbered C8 to C3, C9 to C4, U51 to U3, U52 to U4
Connections:
- net labels added: D+, D-, USB_D+, USB_D-
- wire segments 45 -> 49
- no-connect marks 3 -> 1
Changed lines of the file:
@@
 $EndDescr
 $Comp
-L Regulator_Switching:LM3670MF U52
+L Regulator_Switching:LM3670MF U4
 U 1 1 5F788F1B
 P 5500 3550
-F 0 "U52" H 5500 3875 50  0000 C CNN
+F 0 "U4" H 5500 3875 50  0000 C CNN
 F 1 "LM3671MF-3.3" H 5500 3784 50  0000 C CNN
 F 2 "Package_TO_SOT_SMD:TSOT-23-5" H 5550 3300 50  0001 L CNN
@@
 	5200 3450 5075 3450
 $Comp
-L Device:C C9
+L Device:C C4
 U 1 1 5F78C119
 P 6725 3750
-F 0 "C9" H 6840 3796 50  0000 L CNN
+F 0 "C4" H 6840 3796 50  0000 L CNN
 F 1 "10uF" H 6840 3705 50  0000 L CNN
 F 2 "" H 6763 3600 50  0001 C CNN
@@
 	6475 3450 6725 3450
 $Comp
-L power:GND #PWR020
+L power:GND #PWR09
 U 1 1 5F78F1EA
 P 5500 3975
-F 0 "#PWR020" H 5500 3725 50  0001 C CNN
+F 0 "#PWR09" H 5500 3725 50  0001 C CNN
 F 1 "GND" H 5505 3802 50  0000 C CNN
 F 2 "" H 5500 3975 50  0001 C CNN
@@
 $EndComp
 $Comp
-L local:P-FET U51
+L local:P-FET U3
 U 1 1 5F8BAAF4
 P 3925 3500
-F 0 "U51" H 3925 3815 50  0000 C CNN
+F 0 "U3" H 3925 3815 50  0000 C CNN
 F 1 "P-FET" H 3925 3724 50  0000 C CNN
 F 2 "" H 4125 3900 50  0001 C CNN
@@
 Wire Wire Line
 	3525 3550 3625 3550
-NoConn ~ 3625 2200
-NoConn ~ 3725 2200
 $Comp
 L pspice:DIODE D1
@@
 	4925 3900 4925 3975
 $Comp
-L Device:C C8
+L Device:C C3
 U 1 1 5F789842
 P 4925 3750
-F 0 "C8" H 4725 3750 50  0000 L CNN
+F 0 "C3" H 4725 3750 50  0000 L CNN
 F 1 "4.7uF" H 4700 3650 50  0000 L CNN
 F 2 "" H 4963 3600 50  0001 C CNN
@@
 	4925 3975 5150 3975
 Wire Wire Line
-	3825 2200 3825 2375
-Wire Wire Line
-	3825 2375 4500 2375
-Wire Wire Line
-	4500 2375 4500 3975
+	3825 2200 3825 2225
+Wire Wire Line
+	3825 2225 4500 2225
+Wire Wire Line
+	4500 2225 4500 3975
 Wire Wire Line
 	6725 3450 7325 3450
 Text Label 7000 3450 0    50   ~ 0
 3.3V
-Text Label 3525 2275 3    50   ~ 0
+Text Label 3525 2200 3    50   ~ 0
 5V
 Wire Wire Line
@@
 	5075 3450 4925 3450
 $Comp
-L power:GND #PWR019
+L power:GND #PWR08
 U 1 1 5F8DC955
 P 3300 2025
-F 0 "#PWR019" H 3300 1775 50  0001 C CNN
+F 0 "#PWR08" H 3300 1775 50  0001 C CNN
 F 1 "GND" H 3305 1852 50  0000 C CNN
 F 2 "" H 3300 2025 50  0001 C CNN
@@
 	4575 3450 4925 3450
 NoConn ~ 4225 3550
+Text Label 3625 2300 1    50   ~ 0
+D-
+Text Label 3725 2300 1    50   ~ 0
+D+
+Wire Wire Line
+	3625 2375 2125 2375
+Wire Wire Line
+	3625 2200 3625 2375
+Wire Wire Line
+	3725 2475 2125 2475
+Wire Wire Line
+	3725 2200 3725 2475
+Text HLabel 2125 2375 0    50   Input ~ 0
+USB_D-
+Text HLabel 2125 2475 0    50   Input ~ 0
+USB_D+
 $EndSCHEMATC

Commit message: Adds IrDA transceiver
Parts:
- renumbered C3 to C4, C4 to C5, R1 to R2, R2 to R3
Changed lines of the file:
@@
 	5200 3450 5075 3450
 $Comp
-L Device:C C4
+L Device:C C5
 U 1 1 5F78C119
 P 6725 3750
-F 0 "C4" H 6840 3796 50  0000 L CNN
+F 0 "C5" H 6840 3796 50  0000 L CNN
 F 1 "10uF" H 6840 3705 50  0000 L CNN
 F 2 "" H 6763 3600 50  0001 C CNN
@@
 	6475 3450 6725 3450
 $Comp
-L power:GND #PWR09
+L power:GND #PWR010
 U 1 1 5F78F1EA
 P 5500 3975
-F 0 "#PWR09" H 5500 3725 50  0001 C CNN
+F 0 "#PWR010" H 5500 3725 50  0001 C CNN
 F 1 "GND" H 5505 3802 50  0000 C CNN
 F 2 "" H 5500 3975 50  0001 C CNN
@@
 	3625 3450 3400 3450
 $Comp
-L Device:R R1
+L Device:R R2
 U 1 1 5F8BFEFE
 P 3525 3825
-F 0 "R1" H 3595 3871 50  0000 L CNN
+F 0 "R2" H 3595 3871 50  0000 L CNN
 F 1 "10K" H 3595 3780 50  0000 L CNN
 F 2 "" V 3455 3825 50  0001 C CNN
@@
 	4925 3900 4925 3975
 $Comp
-L Device:C C3
+L Device:C C4
 U 1 1 5F789842
 P 4925 3750
-F 0 "C3" H 4725 3750 50  0000 L CNN
+F 0 "C4" H 4725 3750 50  0000 L CNN
 F 1 "4.7uF" H 4700 3650 50  0000 L CNN
 F 2 "" H 4963 3600 50  0001 C CNN
@@
 	5075 3450 4925 3450
 $Comp
-L power:GND #PWR08
+L power:GND #PWR09
 U 1 1 5F8DC955
 P 3300 2025
-F 0 "#PWR08" H 3300 1775 50  0001 C CNN
+F 0 "#PWR09" H 3300 1775 50  0001 C CNN
 F 1 "GND" H 3305 1852 50  0000 C CNN
 F 2 "" H 3300 2025 50  0001 C CNN
@@
 $EndComp
 $Comp
-L Device:R R2
+L Device:R R3
 U 1 1 5F2BAEAD
 P 5150 3825
-F 0 "R2" H 5220 3871 50  0000 L CNN
+F 0 "R3" H 5220 3871 50  0000 L CNN
 F 1 "100K" H 5220 3780 50  0000 L CNN
 F 2 "" V 5080 3825 50  0001 C CNN

Commit message: Adds power switch
Parts:
- added S?: JS202011SCQN, digikey-footprints:Switch_Slide_JS202011SCQN, symbol dk_Slide-Switches:JS202011SCQN
Connections:
- wire segments 49 -> 54
Other:
- moved on the sheet: BT1
Changed lines of the file:
@@
 L Device:Battery BT1
 U 1 1 5F7915DC
-P 2075 3450
-F 0 "BT1" V 1925 3375 50  0000 L CNN
-F 1 "2 x 1.5V AA" V 2225 3225 50  0000 L CNN
-F 2 "" V 2075 3510 50  0001 C CNN
-F 3 "~" V 2075 3510 50  0001 C CNN
-	1    2075 3450
+P 2075 3350
+F 0 "BT1" V 1925 3275 50  0000 L CNN
+F 1 "2 x 1.5V AA" V 2225 3125 50  0000 L CNN
+F 2 "" V 2075 3410 50  0001 C CNN
+F 3 "~" V 2075 3410 50  0001 C CNN
+	1    2075 3350
 	0    1    -1   0
 $EndComp
@@
 	4225 3450 4300 3450
 Connection ~ 4300 3450
-Text Label 2475 3450 2    50   ~ 0
+Text Label 2450 3350 2    50   ~ 0
 6V
 $Comp
@@
 $EndComp
 Wire Wire Line
-	1825 3450 1875 3450
+	1825 3350 1875 3350
 Wire Wire Line
 	4925 3600 4925 3450
@@
 $EndComp
 Wire Wire Line
-	3525 2200 3525 2825
-Wire Wire Line
 	3750 2825 3525 2825
-Connection ~ 3525 2825
-Wire Wire Line
-	3525 2825 3525 3550
+Wire Wire Line
+	3525 2825 3525 3050
 Wire Wire Line
 	4150 2825 4300 2825
@@
 Wire Wire Line
 	1875 3975 1825 3975
-Text HLabel 1825 2925 2    50   Output ~ 0
+Text HLabel 1825 2825 2    50   Output ~ 0
 BAT_LVL
 Wire Wire Line
-	1825 3975 1825 3450
+	1825 3975 1825 3350
 Connection ~ 3525 3975
 Wire Wire Line
-	2275 3450 3000 3450
-Wire Wire Line
-	1825 3450 1825 2925
-Connection ~ 1825 3450
+	1825 3350 1825 2825
+Connection ~ 1825 3350
 Text HLabel 7325 3025 2    50   UnSpc ~ 0
 U_PWR
@@
 Text HLabel 2125 2475 0    50   Input ~ 0
 USB_D+
+$Comp
+L dk_Slide-Switches:JS202011SCQN S?
+U 1 1 5F865FA4
+P 2725 3150
+F 0 "S?" H 2700 2875 50  0000 C CNN
+F 1 "JS202011SCQN" H 2700 3550 50  0000 C CNN
+F 2 "digikey-footprints:Switch_Slide_JS202011SCQN" H 2925 3350 50  0001 L CNN
+F 3 "https://www.ckswitches.com/media/1422/js.pdf" H 2925 3450 60  0001 L CNN
+F 4 "401-2002-1-ND" H 2925 3550 60  0001 L CNN "Digi-Key_PN"
+F 5 "JS202011SCQN" H 2925 3650 60  0001 L CNN "MPN"
+F 6 "Switches" H 2925 3750 60  0001 L CNN "Category"
+F 7 "Slide Switches" H 2925 3850 60  0001 L CNN "Family"
+F 8 "https://www.ckswitches.com/media/1422/js.pdf" H 2925 3950 60  0001 L CNN "DK_Datasheet_Link"
+F 9 "/product-detail/en/c-k/JS202011SCQN/401-2002-1-ND/1640098" H 2925 4050 60  0001 L CNN "DK_Detail_Page"
+F 10 "SWITCH SLIDE DPDT 300MA 6V" H 2925 4150 60  0001 L CNN "Description"
+F 11 "C&K" H 2925 4250 60  0001 L CNN "Manufacturer"
+F 12 "Active" H 2925 4350 60  0001 L CNN "Status"
+	1    2725 3150
+	1    0    0    1
+$EndComp
+Wire Wire Line
+	2925 3450 3000 3450
+Wire Wire Line
+	2275 3350 2525 3350
+Wire Wire Line
+	2925 3050 3525 3050
+Connection ~ 3525 3050
+Wire Wire Line
+	3525 3050 3525 3550
+Wire Wire Line
+	3525 2200 3525 2575
+Wire Wire Line
+	3525 2575 2525 2575
+Wire Wire Line
+	2525 2575 2525 2950
 $EndSCHEMATC

Commit message: Adds GPIO expansion port
Parts:
- gave numbers to parts that had none: 1
- renumbered C4 to C5, C5 to C6, J3 to J4, R2 to R4, R3 to R5
Connections:
- no-connect marks 1 -> 3
Changed lines of the file:
@@
 	5200 3450 5075 3450
 $Comp
-L Device:C C5
+L Device:C C6
 U 1 1 5F78C119
 P 6725 3750
-F 0 "C5" H 6840 3796 50  0000 L CNN
+F 0 "C6" H 6840 3796 50  0000 L CNN
 F 1 "10uF" H 6840 3705 50  0000 L CNN
 F 2 "" H 6763 3600 50  0001 C CNN
@@
 	6475 3450 6725 3450
 $Comp
-L power:GND #PWR010
+L power:GND #PWR015
 U 1 1 5F78F1EA
 P 5500 3975
-F 0 "#PWR010" H 5500 3725 50  0001 C CNN
+F 0 "#PWR015" H 5500 3725 50  0001 C CNN
 F 1 "GND" H 5505 3802 50  0000 C CNN
 F 2 "" H 5500 3975 50  0001 C CNN
@@
 	6275 3975 6725 3975
 $Comp
-L dk_USB-DVI-HDMI-Connectors:UE27AC54100 J3
+L dk_USB-DVI-HDMI-Connectors:UE27AC54100 J4
 U 1 1 5F8B701D
 P 3625 1900
-F 0 "J3" V 3692 2253 60  0000 L CNN
+F 0 "J4" V 3692 2253 60  0000 L CNN
 F 1 "UE27AC54100" V 3798 2253 60  0000 L CNN
 F 2 "digikey-footprints:USB_A_Female_UE27AC54100" H 3825 2100 60  0001 L CNN
@@
 	3625 3450 3400 3450
 $Comp
-L Device:R R2
+L Device:R R4
 U 1 1 5F8BFEFE
 P 3525 3825
-F 0 "R2" H 3595 3871 50  0000 L CNN
+F 0 "R4" H 3595 3871 50  0000 L CNN
 F 1 "10K" H 3595 3780 50  0000 L CNN
 F 2 "" V 3455 3825 50  0001 C CNN
@@
 	4925 3900 4925 3975
 $Comp
-L Device:C C4
+L Device:C C5
 U 1 1 5F789842
 P 4925 3750
-F 0 "C4" H 4725 3750 50  0000 L CNN
+F 0 "C5" H 4725 3750 50  0000 L CNN
 F 1 "4.7uF" H 4700 3650 50  0000 L CNN
 F 2 "" H 4963 3600 50  0001 C CNN
@@
 	5075 3450 4925 3450
 $Comp
-L power:GND #PWR09
+L power:GND #PWR014
 U 1 1 5F8DC955
 P 3300 2025
-F 0 "#PWR09" H 3300 1775 50  0001 C CNN
+F 0 "#PWR014" H 3300 1775 50  0001 C CNN
 F 1 "GND" H 3305 1852 50  0000 C CNN
 F 2 "" H 3300 2025 50  0001 C CNN
@@
 $EndComp
 $Comp
-L Device:R R3
+L Device:R R5
 U 1 1 5F2BAEAD
 P 5150 3825
-F 0 "R3" H 5220 3871 50  0000 L CNN
+F 0 "R5" H 5220 3871 50  0000 L CNN
 F 1 "100K" H 5220 3780 50  0000 L CNN
 F 2 "" V 5080 3825 50  0001 C CNN
@@
 USB_D+
 $Comp
-L dk_Slide-Switches:JS202011SCQN S?
+L dk_Slide-Switches:JS202011SCQN S9
 U 1 1 5F865FA4
 P 2725 3150
-F 0 "S?" H 2700 2875 50  0000 C CNN
+F 0 "S9" H 2700 2875 50  0000 C CNN
 F 1 "JS202011SCQN" H 2700 3550 50  0000 C CNN
 F 2 "digikey-footprints:Switch_Slide_JS202011SCQN" H 2925 3350 50  0001 L CNN
@@
 Wire Wire Line
 	2525 2575 2525 2950
+NoConn ~ 2925 2850
+NoConn ~ 2925 3250
 $EndSCHEMATC
