File: kicad/power.sch (KiCad schematic (older format))
At the start: 13 parts, among them J4 UE27AC54100, U3 P-FET, U4 LM3671MF-3.3

Commit message: Adds AA battery holders
Parts:
- BT1, BT2: footprint (none) -> Battery:BatteryHolder_MPD_BC2AAPC_2xAA
- C5, C6: footprint (none) -> Capacitor_SMD:C_0805_2012Metric_Pad1.15x1.40mm_HandSolder
- R4, R5: footprint (none) -> Resistor_SMD:R_0805_2012Metric_Pad1.15x1.40mm_HandSolder
- U3: footprint (none) -> local:SOIC-8_3.9x4.9mm_P1.27mm_widepads
Changed lines of the file:
@@
 F 0 "C6" H 6840 3796 50  0000 L CNN
 F 1 "10uF" H 6840 3705 50  0000 L CNN
-F 2 "" H 6763 3600 50  0001 C CNN
+F 2 "Capacitor_SMD:C_0805_2012Metric_Pad1.15x1.40mm_HandSolder" H 6763 3600 50  0001 C CNN
 F 3 "~" H 6725 3750 50  0001 C CNN
 	1    6725 3750
@@
 F 0 "BT1" V 1925 3275 50  0000 L CNN
 F 1 "2 x 1.5V AA" V 2225 3125 50  0000 L CNN
-F 2 "" V 2075 3410 50  0001 C CNN
+F 2 "Battery:BatteryHolder_MPD_BC2AAPC_2xAA" V 2075 3410 50  0001 C CNN
 F 3 "~" V 2075 3410 50  0001 C CNN
 	1    2075 3350
@@
 F 0 "U3" H 3925 3815 50  0000 C CNN
 F 1 "P-FET" H 3925 3724 50  0000 C CNN
-F 2 "" H 4125 3900 50  0001 C CNN
+F 2 "local:SOIC-8_3.9x4.9mm_P1.27mm_widepads" H 4125 3900 50  0001 C CNN
 F 3 "https://www.diodes.com/assets/Datasheets/DMP3085LSD.pdf" H 4125 3900 50  0001 C CNN
 	1    3925 3500
@@
 F 0 "R4" H 3595 3871 50  0000 L CNN
 F 1 "10K" H 3595 3780 50  0000 L CNN
-F 2 "" V 3455 3825 50  0001 C CNN
+F 2 "Resistor_SMD:R_0805_2012Metric_Pad1.15x1.40mm_HandSolder" V 3455 3825 50  0001 C CNN
 F 3 "~" H 3525 3825 50  0001 C CNN
 	1    3525 3825
@@
 F 0 "C5" H 4725 3750 50  0000 L CNN
 F 1 "4.7uF" H 4700 3650 50  0000 L CNN
-F 2 "" H 4963 3600 50  0001 C CNN
+F 2 "Capacitor_SMD:C_0805_2012Metric_Pad1.15x1.40mm_HandSolder" H 4963 3600 50  0001 C CNN
 F 3 "~" H 4925 3750 50  0001 C CNN
 	1    4925 3750
@@
 F 0 "R5" H 5220 3871 50  0000 L CNN
 F 1 "100K" H 5220 3780 50  0000 L CNN
-F 2 "" V 5080 3825 50  0001 C CNN
+F 2 "Resistor_SMD:R_0805_2012Metric_Pad1.15x1.40mm_HandSolder" V 5080 3825 50  0001 C CNN
 F 3 "~" H 5150 3825 50  0001 C CNN
 	1    5150 3825
@@
 F 0 "BT2" V 1925 3925 50  0000 L CNN
 F 1 "2 x 1.5V AA" V 2225 3750 50  0000 L CNN
-F 2 "" V 2075 4035 50  0001 C CNN
+F 2 "Battery:BatteryHolder_MPD_BC2AAPC_2xAA" V 2075 4035 50  0001 C CNN
 F 3 "~" V 2075 4035 50  0001 C CNN
 	1    2075 3975

Commit message: Adds AVR/PDI header footprint
Parts:
- D1, D2: value 1N4007 -> MRA4007; footprint (none) -> Diode_SMD:D_SMA_Handsoldering
- renumbered S9 to S1
Changed lines of the file:
@@
 P 3200 3450
 F 0 "D1" H 3200 3715 50  0000 C CNN
-F 1 "1N4007" H 3200 3624 50  0000 C CNN
-F 2 "" H 3200 3450 50  0001 C CNN
-F 3 "~" H 3200 3450 50  0001 C CNN
+F 1 "MRA4007" H 3200 3624 50  0000 C CNN
+F 2 "Diode_SMD:D_SMA_Handsoldering" H 3200 3450 50  0001 C CNN
+F 3 "https://www.onsemi.com/pub/Collateral/MRA4003T3-D.PDF" H 3200 3450 50  0001 C CNN
 	1    3200 3450
 	1    0    0    -1
@@
 P 3950 2825
 F 0 "D2" H 3950 3090 50  0000 C CNN
-F 1 "1N4007" H 3950 2999 50  0000 C CNN
-F 2 "" H 3950 2825 50  0001 C CNN
-F 3 "~" H 3950 2825 50  0001 C CNN
+F 1 "MRA4007" H 3950 2999 50  0000 C CNN
+F 2 "Diode_SMD:D_SMA_Handsoldering" H 3950 2825 50  0001 C CNN
+F 3 "https://www.onsemi.com/pub/Collateral/MRA4003T3-D.PDF" H 3950 2825 50  0001 C CNN
 	1    3950 2825
 	1    0    0    -1
@@
 USB_D+
 $Comp
-L dk_Slide-Switches:JS202011SCQN S9
+L dk_Slide-Switches:JS202011SCQN S1
 U 1 1 5F865FA4
 P 2725 3150
-F 0 "S9" H 2700 2875 50  0000 C CNN
+F 0 "S1" H 2700 2875 50  0000 C CNN
 F 1 "JS202011SCQN" H 2700 3550 50  0000 C CNN
 F 2 "digikey-footprints:Switch_Slide_JS202011SCQN" H 2925 3350 50  0001 L CNN

Commit message: Adds inductor datasheet
Parts:
- removed R5: 100K, Resistor_SMD:R_0805_2012Metric_Pad1.15x1.40mm_HandSolder, symbol Device:R
- L1: value 2.2uH -> 10uH
Connections:
- wire segments 54 -> 51
Changed lines of the file:
@@
 P 6225 3450
 F 0 "L1" V 6044 3450 50  0000 C CNN
-F 1 "2.2uH" V 6135 3450 50  0000 C CNN
+F 1 "10uH" V 6135 3450 50  0000 C CNN
 F 2 "" H 6225 3450 50  0001 C CNN
-F 3 "~" H 6225 3450 50  0001 C CNN
+F 3 "http://products.sumida.com/products/pdf/CDRH5D18,5D18BHP.pdf" H 6225 3450 50  0001 C CNN
 	1    6225 3450
 	0    1    1    0
@@
 Connection ~ 4925 3975
 Wire Wire Line
-	4925 3975 5150 3975
-Wire Wire Line
 	3825 2200 3825 2225
 Wire Wire Line
@@
 	4300 2825 4300 3450
 Wire Wire Line
-	5200 3550 5150 3550
-Wire Wire Line
 	5075 3550 5075 3450
 Connection ~ 5075 3450
@@
 	1    0    0    -1
 $EndComp
-$Comp
-L Device:R R5
-U 1 1 5F2BAEAD
-P 5150 3825
-F 0 "R5" H 5220 3871 50  0000 L CNN
-F 1 "100K" H 5220 3780 50  0000 L CNN
-F 2 "Resistor_SMD:R_0805_2012Metric_Pad1.15x1.40mm_HandSolder" V 5080 3825 50  0001 C CNN
-F 3 "~" H 5150 3825 50  0001 C CNN
-	1    5150 3825
-	1    0    0    -1
-$EndComp
-Connection ~ 5150 3975
-Wire Wire Line
-	5150 3975 5500 3975
-Wire Wire Line
-	5150 3675 5150 3550
-Connection ~ 5150 3550
-Wire Wire Line
-	5150 3550 5075 3550
 Wire Wire Line
 	4575 3450 4575 3025
@@
 NoConn ~ 2925 2850
 NoConn ~ 2925 3250
+Wire Wire Line
+	4925 3975 5500 3975
+Wire Wire Line
+	5075 3550 5200 3550
 $EndSCHEMATC

Commit message: Adds inductor footprint
Parts:
- L1: footprint (none) -> local:CDRH5D18NP
Connections:
- wire segments 51 -> 53
- no-connect marks 3 -> 2
Changed lines of the file:
@@
 F 0 "L1" V 6044 3450 50  0000 C CNN
 F 1 "10uH" V 6135 3450 50  0000 C CNN
-F 2 "" H 6225 3450 50  0001 C CNN
+F 2 "local:CDRH5D18NP" H 6225 3450 50  0001 C CNN
 F 3 "http://products.sumida.com/products/pdf/CDRH5D18,5D18BHP.pdf" H 6225 3450 50  0001 C CNN
 	1    6225 3450
@@
 Wire Wire Line
 	4575 3450 4925 3450
-NoConn ~ 4225 3550
 Text Label 3625 2300 1    50   ~ 0
 D-
@@
 Wire Wire Line
 	5075 3550 5200 3550
+Wire Wire Line
+	4225 3550 4300 3550
+Wire Wire Line
+	4300 3550 4300 3450
 $EndSCHEMATC

Commit message: Switches battery holders and adds switch footprint
Parts:
- BT1, BT2: footprint Battery:BatteryHolder_MPD_BC2AAPC_2xAA -> Battery:BatteryHolder_MPD_BC12AAPC_2xAA
- S1: footprint digikey-footprints:Switch_Slide_JS202011SCQN -> local:JS202011AQN_THT_DPDT
Changed lines of the file:
@@
 F 0 "BT1" V 1925 3275 50  0000 L CNN
 F 1 "2 x 1.5V AA" V 2225 3125 50  0000 L CNN
-F 2 "Battery:BatteryHolder_MPD_BC2AAPC_2xAA" V 2075 3410 50  0001 C CNN
+F 2 "Battery:BatteryHolder_MPD_BC12AAPC_2xAA" V 2075 3410 50  0001 C CNN
 F 3 "~" V 2075 3410 50  0001 C CNN
 	1    2075 3350
@@
 F 0 "BT2" V 1925 3925 50  0000 L CNN
 F 1 "2 x 1.5V AA" V 2225 3750 50  0000 L CNN
-F 2 "Battery:BatteryHolder_MPD_BC2AAPC_2xAA" V 2075 4035 50  0001 C CNN
+F 2 "Battery:BatteryHolder_MPD_BC12AAPC_2xAA" V 2075 4035 50  0001 C CNN
 F 3 "~" V 2075 4035 50  0001 C CNN
 	1    2075 3975
@@
 F 0 "S1" H 2700 2875 50  0000 C CNN
 F 1 "JS202011SCQN" H 2700 3550 50  0000 C CNN
-F 2 "digikey-footprints:Switch_Slide_JS202011SCQN" H 2925 3350 50  0001 L CNN
+F 2 "local:JS202011AQN_THT_DPDT" H 2925 3350 50  0001 L CNN
 F 3 "https://www.ckswitches.com/media/1422/js.pdf" H 2925 3450 60  0001 L CNN
 F 4 "401-2002-1-ND" H 2925 3550 60  0001 L CNN "Digi-Key_PN"

Commit message: Adds board outline
Parts:
- added unit 2 of U3
Connections:
- wire segments 53 -> 57
- no-connect marks 2 -> 4
Changed lines of the file:
@@
 Wire Wire Line
 	4300 3550 4300 3450
+$Comp
+L local:P-FET U?
+U 2 1 5F952E8F
+P 3925 4300
+AR Path="/6011206E/5F952E8F" Ref="U?"  Part="2"
+AR Path="/5F785555/5F952E8F" Ref="U3"  Part="2"
+F 0 "U3" H 3675 4500 50  0000 C CNN
+F 1 "P-FET" V 3925 4300 50  0000 C CNN
+F 2 "local:SOIC-8_3.9x4.9mm_P1.27mm_widepads" H 4125 4700 50  0001 C CNN
+F 3 "https://www.diodes.com/assets/Datasheets/DMP3085LSD.pdf" H 4125 4700 50  0001 C CNN
+	2    3925 4300
+	1    0    0    -1
+$EndComp
+NoConn ~ 4225 4350
+NoConn ~ 4225 4250
+Wire Wire Line
+	3625 4350 3625 4300
+Wire Wire Line
+	3625 4300 3525 4300
+Connection ~ 3625 4300
+Wire Wire Line
+	3625 4300 3625 4250
+Wire Wire Line
+	3525 4300 3525 3975
 $EndSCHEMATC

Commit message: Starts matrix driver component layout
Parts:
- U3: footprint local:SOIC-8_3.9x4.9mm_P1.27mm_widepads -> Package_SO:SOIC-8_3.9x4.9mm_P1.27mm
Changed lines of the file:
@@
 F 0 "U3" H 3925 3815 50  0000 C CNN
 F 1 "P-FET" H 3925 3724 50  0000 C CNN
-F 2 "local:SOIC-8_3.9x4.9mm_P1.27mm_widepads" H 4125 3900 50  0001 C CNN
+F 2 "Package_SO:SOIC-8_3.9x4.9mm_P1.27mm" H 4125 3900 50  0001 C CNN
 F 3 "https://www.diodes.com/assets/Datasheets/DMP3085LSD.pdf" H 4125 3900 50  0001 C CNN
 	1    3925 3500
@@
 F 0 "U3" H 3675 4500 50  0000 C CNN
 F 1 "P-FET" V 3925 4300 50  0000 C CNN
-F 2 "local:SOIC-8_3.9x4.9mm_P1.27mm_widepads" H 4125 4700 50  0001 C CNN
+F 2 "Package_SO:SOIC-8_3.9x4.9mm_P1.27mm" H 4125 4700 50  0001 C CNN
 F 3 "https://www.diodes.com/assets/Datasheets/DMP3085LSD.pdf" H 4125 4700 50  0001 C CNN
 	2    3925 4300

Commit message: Added power plane and reassigned pinout
Parts:
- removed D1, D2: MRA4007, Diode_SMD:D_SMA_Handsoldering, symbol pspice:DIODE
- added D1, D2: MRA4003T3G, Diode_SMD:D_SMA, symbol Diode:MRA4003T3G
Changed lines of the file:
@@
 Wire Wire Line
 	3525 3550 3625 3550
-$Comp
-L pspice:DIODE D1
-U 1 1 5F8CC172
-P 3200 3450
-F 0 "D1" H 3200 3715 50  0000 C CNN
-F 1 "MRA4007" H 3200 3624 50  0000 C CNN
-F 2 "Diode_SMD:D_SMA_Handsoldering" H 3200 3450 50  0001 C CNN
-F 3 "https://www.onsemi.com/pub/Collateral/MRA4003T3-D.PDF" H 3200 3450 50  0001 C CNN
-	1    3200 3450
-	1    0    0    -1
-$EndComp
 Wire Wire Line
 	1825 3350 1875 3350
@@
 	4500 3975 4925 3975
 Connection ~ 3525 3550
-$Comp
-L pspice:DIODE D2
-U 1 1 5F8D97D5
-P 3950 2825
-F 0 "D2" H 3950 3090 50  0000 C CNN
-F 1 "MRA4007" H 3950 2999 50  0000 C CNN
-F 2 "Diode_SMD:D_SMA_Handsoldering" H 3950 2825 50  0001 C CNN
-F 3 "https://www.onsemi.com/pub/Collateral/MRA4003T3-D.PDF" H 3950 2825 50  0001 C CNN
-	1    3950 2825
-	1    0    0    -1
-$EndComp
 Wire Wire Line
 	3750 2825 3525 2825
@@
 	3525 2825 3525 3050
 Wire Wire Line
-	4150 2825 4300 2825
+	4050 2825 4300 2825
 Wire Wire Line
 	4300 2825 4300 3450
@@
 $EndComp
 Wire Wire Line
-	2925 3450 3000 3450
+	2925 3450 3100 3450
 Wire Wire Line
 	2275 3350 2525 3350
@@
 Wire Wire Line
 	3525 4300 3525 3975
+$Comp
+L Diode:MRA4003T3G D1
+U 1 1 5FBA69DF
+P 3250 3450
+F 0 "D1" H 3250 3233 50  0000 C CNN
+F 1 "MRA4003T3G" H 3250 3324 50  0000 C CNN
+F 2 "Diode_SMD:D_SMA" H 3250 3275 50  0001 C CNN
+F 3 "http://www.onsemi.com/pub_link/Collateral/MRA4003T3-D.PDF" H 3250 3450 50  0001 C CNN
+	1    3250 3450
+	-1   0    0    1
+$EndComp
+$Comp
+L Diode:MRA4003T3G D2
+U 1 1 5FBAF34B
+P 3900 2825
+F 0 "D2" H 3900 2608 50  0000 C CNN
+F 1 "MRA4003T3G" H 3900 2699 50  0000 C CNN
+F 2 "Diode_SMD:D_SMA" H 3900 2650 50  0001 C CNN
+F 3 "http://www.onsemi.com/pub_link/Collateral/MRA4003T3-D.PDF" H 3900 2825 50  0001 C CNN
+	1    3900 2825
+	-1   0    0    1
+$EndComp
 $EndSCHEMATC
