File: kicad/handheld.kicad_pcb (KiCad board)
At the start: 4 copper layers, 240 x 77.7 mm, 113 parts, among them J1 Conn_01x08, J2 61300311121, J3 AVR-PDI-6, J4 UE27AC54100, Q1 PN2222A, SW1 HOLD, SW10 SELECT, SW2 PAUSE, SW3 SDROP, SW4 HDROP, SW5 ROTR, SW6 RIGHT, SW7 ROTL, SW8 RIGHT, SW9 START, U1 TFBS4711, U10 DMN601, U11 NSI45015, U12 SN54LV574, U13 P-FET, U14 NSI45015, U15 DMN601, U16 NSI45015, U17 NSI45015, U18 DMN601, U19 P-FET, U2 ATxmega64C3-AU, U20 NSI45015, U21 74HCT595, U22 NSI45015, U23 DMN601, U24 NSI45015, U25 P-FET, U26 NSI45015, U27 DMN601, U28 NSI45015, U29 SN54LV574, U3 P-FET, U30 NSI45015, U31 DMN601, U32 NSI45015, U33 P-FET, U34 NSI45015, U35 DMN601, U36 NSI45015, U37 NSI45015, U38 P-FET, U39 DMN601, U4 LM3671MF-3.3, U40 NSI45015, U41 NSI45015, U42 DMN601, U43 NSI45015, U44 SN54LV574, U45 74HCT595, U46 P-FET, U47 NSI45015, U48 DMN601, U49 NSI45015, U5 NSI45015, U50 NSI45015, U51 DMN601, U52 P-FET, U53 NSI45015, U54 SN74LVC1G08DBVR, U55 SN74LVC1G08DBVR, U56 SN74LVC1G08DBVR, U57 SN74LVC1G08DBVR, U6 P-FET, U7 DMN601, U8 NSI45015, U9 NSI45015

Commit message: Switched to registers with clear
Also added the mountng holes as annotated symbols with footprints.
Parts:
- added G***: LOGO, arrow:arraw_6mm, F.Cu at (45.5, 98.0)
- added G***: LOGO, arrow:arraw_6mm, F.Cu at (53.6, 85.5)
- added G***: LOGO, arrow:arraw_6mm, F.Cu at (83.0, 105.1)
- added G***: LOGO, arrow:arraw_6mm, F.Cu at (74.9, 117.7)
- added H1: MountingHole, MountingHole:MountingHole_3.2mm_M3, F.Cu at (47.4, 73.6)
- added H2: MountingHole, MountingHole:MountingHole_3.2mm_M3, F.Cu at (257.4, 73.6)
- added H3: MountingHole, MountingHole:MountingHole_3.2mm_M3, F.Cu at (47.4, 129.6)
- added H4: MountingHole, MountingHole:MountingHole_3.2mm_M3, F.Cu at (257.4, 129.6)
- added H5: MountingHole, MountingHole:MountingHole_3.2mm_M3, F.Cu at (133.4, 101.6)
- added H6: MountingHole, MountingHole:MountingHole_3.2mm_M3, F.Cu at (171.3, 101.6)
- added REF**: OSHW-Logo_5.7x6mm_Copper, Symbol:OSHW-Logo_5.7x6mm_Copper, B.Cu at (265.4, 129.6)
- added REF**: OSHW-Logo_5.7x6mm_Copper, Symbol:OSHW-Logo_5.7x6mm_Copper, F.Cu at (39.4, 73.6)
- added REF**: OSHW-Logo2_9.8x8mm_SilkScreen, Symbol:OSHW-Logo2_9.8x8mm_SilkScreen, F.Cu at (240.3, 129.6)
- added REF**: KiCad-Logo_6mm_SilkScreen, Symbol:KiCad-Logo_6mm_SilkScreen, F.Cu at (64.3, 129.6)
- U12, U29, U44: value SN54LV574 -> SN74LV573
Connections:
- U12 pad 1: /~OE -> VDD
- U29 pad 1: /~OE -> VDD
- U44 pad 1: /~OE -> VDD
Routing:
- net /~OE: track 157.5 -> 14.0 mm, vias 6 -> 0
- net VDD: track 47.5 -> 63.8 mm, vias 22 -> 23
- net /Matrix Driver/COL15: track 77.0 -> 75.3 mm
- net /Matrix Driver/COL14: track 86.7 -> 85.3 mm

Commit message: Add silkscreen art
Parts:
- added G***: LOGO, warp:warp_B_240mm_mod, B.Cu at (152.3, 100.9)
Routing:
- net GND: track 116.1 -> 114.8 mm
- added copper zone on B.Cu, net GND
Other:
- board text added: "VOL"
- board text removed: "VOLUME"
